Commit message: Update bipedal.urdf
change the amount of max torque

File: bipedal.urdf (robot description, URDF)
Before this commit: robot bipedal, 7 links, 6 joints
Joints:
- joint base_to_left_leg: limit lower=-0.7854 upper=0.7854 effort=50 velocity=5 -> lower=-0.7854 upper=0.7854 effort=5 velocity=5
- joint base_to_right_leg: limit lower=-0.7854 upper=0.7854 effort=50 velocity=5 -> lower=-0.7854 upper=0.7854 effort=5 velocity=5
- joint left_bicep_joint: limit lower=-0.7854 upper=0.7854 effort=50 velocity=5 -> lower=-0.7854 upper=0.7854 effort=5 velocity=5
- joint left_feet_joint: limit lower=-0.7854 upper=0.7854 effort=50 velocity=5 -> lower=-0.7854 upper=0.7854 effort=5 velocity=5
- joint right_bicep_joint: limit lower=-0.7854 upper=0.7854 effort=50 velocity=5 -> lower=-0.7854 upper=0.7854 effort=5 velocity=5
- joint right_feet_joint: limit lower=-0.7854 upper=0.7854 effort=50 velocity=5 -> lower=-0.7854 upper=0.7854 effort=5 velocity=5

Commit message: Update bipedal.urdf
update legs position

File: bipedal.urdf (robot description, URDF)
Before this commit: robot bipedal, 7 links, 6 joints
Joints:
- joint base_to_left_leg: origin xyz=0 0.125 0 rpy=0 0.7854 0 -> xyz=-0.1 0.125 0 rpy=0 0.7854 0
- joint base_to_right_leg: origin xyz=0 -0.125 0 rpy=0 0.7854 0 -> xyz=-0.1 -0.125 0 rpy=0 0.7854 0

Commit message: Update bipedal.urdf

File: bipedal.urdf (robot description, URDF)
Before this commit: robot bipedal, 7 links, 6 joints
Links:
- link base_link: geometry collision box size=0.25 0.25 0.15; visual box size=0.25 0.25 0.15

Commit message: Update bipedal.urdf

File: bipedal.urdf (robot description, URDF)
Before this commit: robot bipedal, 7 links, 6 joints
Joints:
- joint base_to_left_leg: limit lower=-0.7854 upper=0.7854 effort=5 velocity=5 -> lower=-0.7854 upper=0.7854 effort=5 velocity=30
- joint base_to_right_leg: limit lower=-0.7854 upper=0.7854 effort=5 velocity=5 -> lower=-0.7854 upper=0.7854 effort=5 velocity=30
- joint left_bicep_joint: limit lower=-0.7854 upper=0.7854 effort=5 velocity=5 -> lower=-0.7854 upper=0.7854 effort=5 velocity=30
- joint left_feet_joint: limit lower=-0.7854 upper=0.7854 effort=5 velocity=5 -> lower=-0.7854 upper=0.7854 effort=5 velocity=30
- joint right_bicep_joint: limit lower=-0.7854 upper=0.7854 effort=5 velocity=5 -> lower=-0.7854 upper=0.7854 effort=5 velocity=30
- joint right_feet_joint: limit lower=-0.7854 upper=0.7854 effort=5 velocity=5 -> lower=-0.7854 upper=0.7854 effort=5 velocity=30

Commit message: Update bipedal.urdf

File: bipedal.urdf (robot description, URDF)
Before this commit: robot bipedal, 7 links, 6 joints
Joints:
- joint base_to_left_leg: limit lower=-0.7854 upper=0.7854 effort=5 velocity=30 -> lower=-0.7854 upper=0.7854 effort=5 velocity=10
- joint base_to_right_leg: limit lower=-0.7854 upper=0.7854 effort=5 velocity=30 -> lower=-0.7854 upper=0.7854 effort=5 velocity=10
- joint left_bicep_joint: limit lower=-0.7854 upper=0.7854 effort=5 velocity=30 -> lower=-0.7854 upper=0.7854 effort=5 velocity=10
- joint left_feet_joint: limit lower=-0.7854 upper=0.7854 effort=5 velocity=30 -> lower=-0.7854 upper=0.7854 effort=5 velocity=10
- joint right_bicep_joint: limit lower=-0.7854 upper=0.7854 effort=5 velocity=30 -> lower=-0.7854 upper=0.7854 effort=5 velocity=10
- joint right_feet_joint: limit lower=-0.7854 upper=0.7854 effort=5 velocity=30 -> lower=-0.7854 upper=0.7854 effort=5 velocity=10

Commit message: Update bipedal.urdf

File: bipedal.urdf (robot description, URDF)
Before this commit: robot bipedal, 7 links, 6 joints
Joints:
- joint base_to_left_leg: limit lower=-0.7854 upper=0.7854 effort=5 velocity=10 -> lower=-1.57 upper=1.57 effort=5 velocity=10
- joint base_to_right_leg: limit lower=-0.7854 upper=0.7854 effort=5 velocity=10 -> lower=-1.57 upper=1.57 effort=5 velocity=10
- joint left_bicep_joint: limit lower=-0.7854 upper=0.7854 effort=5 velocity=10 -> lower=-1.57 upper=1.57 effort=5 velocity=10
- joint left_feet_joint: limit lower=-0.7854 upper=0.7854 effort=5 velocity=10 -> lower=-1.57 upper=1.57 effort=5 velocity=10
- joint right_bicep_joint: limit lower=-0.7854 upper=0.7854 effort=5 velocity=10 -> lower=-1.57 upper=1.57 effort=5 velocity=10
- joint right_feet_joint: limit lower=-0.7854 upper=0.7854 effort=5 velocity=10 -> lower=-1.57 upper=1.57 effort=5 velocity=10

Commit message: Update bipedal.urdf
change joints limit

File: bipedal.urdf (robot description, URDF)
Before this commit: robot bipedal, 7 links, 6 joints
Joints:
- joint base_to_left_leg: limit lower=-1.57 upper=1.57 effort=5 velocity=10 -> lower=-0.785 upper=0.785 effort=5 velocity=10
- joint base_to_right_leg: limit lower=-1.57 upper=1.57 effort=5 velocity=10 -> lower=-0.785 upper=0.785 effort=5 velocity=10
- joint left_bicep_joint: limit lower=-1.57 upper=1.57 effort=5 velocity=10 -> lower=-0.785 upper=0.785 effort=5 velocity=10
- joint left_feet_joint: limit lower=-1.57 upper=1.57 effort=5 velocity=10 -> lower=-0.785 upper=0.785 effort=5 velocity=10
- joint right_bicep_joint: limit lower=-1.57 upper=1.57 effort=5 velocity=10 -> lower=-0.785 upper=0.785 effort=5 velocity=10
- joint right_feet_joint: limit lower=-1.57 upper=1.57 effort=5 velocity=10 -> lower=-0.785 upper=0.785 effort=5 velocity=10

Commit message: Update bipedal.urdf

File: bipedal.urdf (robot description, URDF)
Before this commit: robot bipedal, 7 links, 6 joints
Joints:
- joint base_to_left_leg: origin xyz=-0.1 0.125 0 rpy=0 0.7854 0 -> xyz=-0.2 0.125 0 rpy=0 0.7854 0
- joint base_to_right_leg: origin xyz=-0.1 -0.125 0 rpy=0 0.7854 0 -> xyz=-0.2 -0.125 0 rpy=0 0.7854 0

Commit message: Update bipedal.urdf

File: bipedal.urdf (robot description, URDF)
Before this commit: robot bipedal, 7 links, 6 joints
Links:
- link base_link: mass 0.2 -> 0.5
Joints:
- joint base_to_left_leg: limit lower=-0.785 upper=0.785 effort=5 velocity=10 -> lower=-0.785 upper=0.785 effort=3 velocity=10
- joint base_to_right_leg: limit lower=-0.785 upper=0.785 effort=5 velocity=10 -> lower=-0.785 upper=0.785 effort=3 velocity=10
- joint left_bicep_joint: limit lower=-0.785 upper=0.785 effort=5 velocity=10 -> lower=-0.785 upper=0.785 effort=3 velocity=10
- joint left_feet_joint: limit lower=-0.785 upper=0.785 effort=5 velocity=10 -> lower=-0.785 upper=0.785 effort=3 velocity=10
- joint right_bicep_joint: limit lower=-0.785 upper=0.785 effort=5 velocity=10 -> lower=-0.785 upper=0.785 effort=3 velocity=10
- joint right_feet_joint: limit lower=-0.785 upper=0.785 effort=5 velocity=10 -> lower=-0.785 upper=0.785 effort=3 velocity=10

Commit message: Update bipedal.urdf

File: bipedal.urdf (robot description, URDF)
Before this commit: robot bipedal, 7 links, 6 joints
Joints:
- joint base_to_left_leg: limit lower=-0.785 upper=0.785 effort=3 velocity=10 -> lower=-0.785 upper=0.785 effort=3 velocity=.5
- joint base_to_right_leg: limit lower=-0.785 upper=0.785 effort=3 velocity=10 -> lower=-0.785 upper=0.785 effort=3 velocity=.5
- joint left_bicep_joint: limit lower=-0.785 upper=0.785 effort=3 velocity=10 -> lower=-0.785 upper=0.785 effort=3 velocity=.5
- joint left_feet_joint: limit lower=-0.785 upper=0.785 effort=3 velocity=10 -> lower=-0.785 upper=0.785 effort=3 velocity=.5
- joint right_bicep_joint: limit lower=-0.785 upper=0.785 effort=3 velocity=10 -> lower=-0.785 upper=0.785 effort=3 velocity=.5
- joint right_feet_joint: limit lower=-0.785 upper=0.785 effort=3 velocity=10 -> lower=-0.785 upper=0.785 effort=3 velocity=.5

Commit message: Update bipedal.urdf

File: bipedal.urdf (robot description, URDF)
Before this commit: robot bipedal, 7 links, 6 joints
Joints:
- joint base_to_left_leg: limit lower=-0.785 upper=0.785 effort=3 velocity=.5 -> lower=-1.57 upper=1.57 effort=3 velocity=.5
- joint base_to_right_leg: limit lower=-0.785 upper=0.785 effort=3 velocity=.5 -> lower=-1.57 upper=1.57 effort=3 velocity=.5
- joint left_bicep_joint: limit lower=-0.785 upper=0.785 effort=3 velocity=.5 -> lower=-1.57 upper=1.57 effort=3 velocity=.5
- joint left_feet_joint: limit lower=-0.785 upper=0.785 effort=3 velocity=.5 -> lower=-1.57 upper=1.57 effort=3 velocity=.5
- joint right_bicep_joint: limit lower=-0.785 upper=0.785 effort=3 velocity=.5 -> lower=-1.57 upper=1.57 effort=3 velocity=.5
- joint right_feet_joint: limit lower=-0.785 upper=0.785 effort=3 velocity=.5 -> lower=-1.57 upper=1.57 effort=3 velocity=.5

Commit message: Update bipedal.urdf

File: bipedal.urdf (robot description, URDF)
Before this commit: robot bipedal, 7 links, 6 joints
Links:
- link base_link: mass 0.5 -> 2.; geometry collision box size=0.15 0.15 0.15; visual box size=0.15 0.15 0.15
- link left_bicep: mass 0.1 -> 0.2; geometry collision box size=0.075 0.075 0.3; visual box size=0.075 0.075 0.3
- link left_feet: mass 0.05 -> 0.1; geometry collision box size=0.125 0.075 0.02; visual box size=0.125 0.075 0.02
- link left_leg: mass 0.1 -> 0.2; geometry collision box size=0.075 0.075 0.3; visual box size=0.075 0.075 0.3
- link right_bicep: mass 0.1 -> 0.2; geometry collision box size=0.075 0.075 0.3; visual box size=0.075 0.075 0.3
- link right_feet: mass 0.05 -> 0.1; geometry collision box size=0.125 0.075 0.02; visual box size=0.125 0.075 0.02
- link right_leg: mass 0.1 -> 0.2; geometry collision box size=0.075 0.075 0.3; visual box size=0.075 0.075 0.3
Joints:
- joint base_to_left_leg: limit lower=-1.57 upper=1.57 effort=3 velocity=.5 -> lower=-0.785 upper=0.785 effort=10 velocity=2; origin xyz=-0.2 0.125 0 rpy=0 0.7854 0 -> xyz=-0.1 0.075 0 rpy=0 0.7854 0
- joint base_to_right_leg: limit lower=-1.57 upper=1.57 effort=3 velocity=.5 -> lower=-0.785 upper=0.785 effort=10 velocity=2; origin xyz=-0.2 -0.125 0 rpy=0 0.7854 0 -> xyz=-0.1 -0.075 0 rpy=0 0.7854 0
- joint left_bicep_joint: limit lower=-1.57 upper=1.57 effort=3 velocity=.5 -> lower=-0.785 upper=0.785 effort=10 velocity=2; origin xyz=0 0.075 -0.15 rpy=0 -1.5708 0 -> xyz=0 0.075 -0.3 rpy=0 -1.5708 0
- joint left_feet_joint: limit lower=-1.57 upper=1.57 effort=3 velocity=.5 -> lower=-0.785 upper=0.785 effort=10 velocity=2; origin xyz=-0.05 0.0375 -0.225 rpy=0 0.7854 0 -> xyz=-0.05 0.0375 -0.3 rpy=0 0.7854 0
- joint right_bicep_joint: limit lower=-1.57 upper=1.57 effort=3 velocity=.5 -> lower=-0.785 upper=0.785 effort=10 velocity=2; origin xyz=0 -0.075 -0.15 rpy=0 -1.5708 0 -> xyz=0 -0.075 -0.3 rpy=0 -1.5708 0
- joint right_feet_joint: limit lower=-1.57 upper=1.57 effort=3 velocity=.5 -> lower=-0.785 upper=0.785 effort=10 velocity=2; origin xyz=-0.05 -0.0375 -0.225 rpy=0 0.7854 0 -> xyz=-0.05 -0.0375 -0.3 rpy=0 0.7854 0
